File: Kicad/lm324_4ch_therm.kicad_pcb (KiCad board)
At the start: 2 copper layers, 24.4 x 20.7 mm, 29 parts, among them J1 NTC50k, J2 supl., J3 NTC50k, J4 NTC50k, J5 NTC50k, J6 Out OC, Q1 MMBT3904, Q2 MMBT3906, U1 LM324

Commit message: Add files via upload
Routing:
- net GND: track 66.8 -> 47.1 mm
Changed lines of the file:
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@@
     (effects (font (size 0.8 0.8) (thickness 0.13)) (justify mirror))
   )
-  (gr_text "GND" (at 117.221 63.373 90) (layer "B.SilkS")
+  (gr_text "GND" (at 117.1448 63.1444 270) (layer "B.SilkS")
     (effects (font (size 0.8 0.8) (thickness 0.13)) (justify mirror))
   )
@@
   (segment (start 129.311 63.774) (end 128.1357 63.774) (width 0.25) (layer "F.Cu") (net 2))
   (via (at 129.3975 47.3814) (size 0.8) (drill 0.4) (layers "F.Cu" "B.Cu") (net 2))
-  (segment (start 129.1966 52.7426) (end 130.302 53.848) (width 0.25) (layer "B.Cu") (net 2))
   (segment (start 127.474 54.8218) (end 127.474 53.1865) (width 0.25) (layer "B.Cu") (net 2))
   (segment (start 123.317 49.407) (end 120.904 49.407) (width 0.25) (layer "B.Cu") (net 2))
   (segment (start 123.317 49.407) (end 124.21 48.514) (width 0.25) (layer "B.Cu") (net 2))
-  (segment (start 127.9179 52.7426) (end 129.1966 52.7426) (width 0.25) (layer "B.Cu") (net 2))
-  (segment (start 130.302 52.1716) (end 132.8676 49.606) (width 0.25) (layer "B.Cu") (net 2))
-  (segment (start 134.874 56.134) (end 134.874 57.3093) (width 0.25) (layer "B.Cu") (net 2))
   (segment (start 134.899 62.5987) (end 135.707 62.5987) (width 0.25) (layer "B.Cu") (net 2))
   (segment (start 133.6591 50.8209) (end 134.874 49.606) (width 0.25) (layer "B.Cu") (net 2))
   (segment (start 134.899 63.774) (end 134.899 62.5987) (width 0.25) (layer "B.Cu") (net 2))
   (segment (start 133.6591 54.9191) (end 133.6591 50.8209) (width 0.25) (layer "B.Cu") (net 2))
-  (segment (start 135.758 58.801) (end 135.758 58.1933) (width 0.25) (layer "B.Cu") (net 2))
   (segment (start 135.707 62.5987) (end 136.0744 62.2313) (width 0.25) (layer "B.Cu") (net 2))
-  (segment (start 130.302 53.848) (end 130.302 52.1716) (width 0.25) (layer "B.Cu") (net 2))
-  (segment (start 117.0218 63.2061) (end 117.0218 55.3868) (width 0.25) (layer "B.Cu") (net 2))
   (segment (start 126.6698 55.626) (end 127.474 54.8218) (width 0.25) (layer "B.Cu") (net 2))
   (segment (start 128.2649 48.514) (end 129.3975 47.3814) (width 0.25) (layer "B.Cu") (net 2))
-  (segment (start 118.745 63.754) (end 117.5697 63.754) (width 0.25) (layer "B.Cu") (net 2))
   (segment (start 136.0744 62.2313) (end 136.0744 59.1174) (width 0.25) (layer "B.Cu") (net 2))
   (segment (start 127.474 53.1865) (end 127.9179 52.7426) (width 0.25) (layer "B.Cu") (net 2))
   (segment (start 124.21 48.514) (end 128.2649 48.514) (width 0.25) (layer "B.Cu") (net 2))
-  (segment (start 117.5697 63.754) (end 117.0218 63.2061) (width 0.25) (layer "B.Cu") (net 2))
-  (segment (start 127.2793 50.2536) (end 127.4949 50.038) (width 0.25) (layer "F.Cu") (net 3))
+  (segment (start 125.0382 50.2536) (end 124.6177 50.6741) (width 0.25) (layer "F.Cu") (net 3))
   (segment (start 122.282 58.536) (end 121.482 58.536) (width 0.25) (layer "F.Cu") (net 3))
-  (segment (start 127.4949 50.038) (end 129.338 50.038) (width 0.25) (layer "F.Cu") (net 3))
   (segment (start 128.8542 51.689) (end 129.6572 50.886) (width 0.32) (layer "F.Cu") (net 3))
   (segment (start 128.378 52.089) (end 128.778 51.689) (width 0.32) (layer "F.Cu") (net 3))
-  (segment (start 129.338 50.038) (end 130.186 50.886) (width 0.25) (layer "F.Cu") (net 3))
+  (segment (start 127.2793 50.2536) (end 125.0382 50.2536) (width 0.25) (layer "F.Cu") (net 3))
+  (segment (start 129.338 50.038) (end 127.4949 50.038) (width 0.25) (layer "F.Cu") (net 3))
+  (segment (start 127.4949 50.038) (end 127.2793 50.2536) (width 0.25) (layer "F.Cu") (net 3))
   (segment (start 123.082 58.536) (end 122.282 58.536) (width 0.25) (layer "F.Cu") (net 3))
   (segment (start 128.378 52.44) (end 128.378 52.089) (width 0.32) (layer "F.Cu") (net 3))
-  (segment (start 124.4259 51.1241) (end 124.4259 51.4213) (width 0.25) (layer "F.Cu") (net 3))
+  (segment (start 124.6177 51.2295) (end 124.4259 51.4213) (width 0.25) (layer "F.Cu") (net 3))
   (segment (start 129.6572 50.886) (end 130.186 50.886) (width 0.32) (layer "F.Cu") (net 3))
   (segment (start 123.882 58.536) (end 123.082 58.536) (width 0.25) (layer "F.Cu") (net 3))
-  (segment (start 125.2964 50.2536) (end 124.4259 51.1241) (width 0.25) (layer "F.Cu") (net 3))
-  (segment (start 127.2793 50.2536) (end 125.2964 50.2536) (width 0.25) (layer "F.Cu") (net 3))
+  (segment (start 130.186 50.886) (end 129.338 50.038) (width 0.25) (layer "F.Cu") (net 3))
   (segment (start 121.423 58.536) (end 118.745 61.214) (width 0.25) (layer "F.Cu") (net 3))
+  (segment (start 124.6177 50.6741) (end 124.6177 51.2295) (width 0.25) (layer "F.Cu") (net 3))
   (segment (start 128.778 51.689) (end 128.8542 51.689) (width 0.32) (layer "F.Cu") (net 3))
   (via (at 124.4259 51.4213) (size 0.8) (drill 0.4) (layers "F.Cu" "B.Cu") (net 3))
